File: cad/BuzzerBox/controller.brd (EAGLE design)
At the start: 100 x 100 mm, 126 parts, among them J1 USB_A_SMT_FEMALE, Q1 BSS138, Q2 BSS138, T1 BC849, T10 BC849, T2 BC849, T3 BC849, T4 BC849, T5 BC849, T6 BC849, T7 BC849, T8 BC849, T9 BC849, U1 ATMEGA328P-AU, Y1 16MHz

Commit message: Add Side-Channel Signal line between uC and RPi
Parts:
- added JP1: (no value), pinhead:2X20
- added Q3: BSS138, SparkFun:SOT23-3
- added R66, R67: 10K, SparkFun-Resistors:0805
- moved RPI-CM1 3.17 mm to (21.0, 87.6)
Connections:
- new net N$47: Q3.2, R67.1, RPI-CM1.55
- net +3V3: now also Q3.1, R67.2
- net +5V: now also R66.2
- net D2: now also Q3.3, R66.1
Routing:
- net USB_N: track 42.1 -> 0.00 mm
- net USB_P: track 41.4 -> 0.00 mm
- net D2: track 0.00 -> 40.4 mm, vias 0 -> 2
- net GND: track 118.0 -> 100.7 mm
- net +3V3: track 70.9 -> 88.0 mm, vias 2 -> 4
- net N$47: track 0.00 -> 11.5 mm
- net +5V: track 602.4 -> 597.3 mm, vias 29 -> 30
- net N$41: track 65.7 -> 63.8 mm
- net SCLPI: track 74.9 -> 73.8 mm
