File: cad/BuzzerBox/controller.sch (EAGLE design)
At the start: 122 parts, among them J1 USB_A_SMT_FEMALE, Q1 BSS138, Q2 BSS138, T1 BC849, T10 BC849, T2 BC849, T3 BC849, T4 BC849, T5 BC849, T6 BC849, T7 BC849, T8 BC849, T9 BC849, U1 ATMEGA328P-AU, Y1 16MHz

Commit message: Add Side-Channel Signal line between uC and RPi
Parts:
- added JP1: (no value), pinhead:PINHD-2X20
- added Q3: BSS138, SparkFun:MOSFET-NCHANNELSMD
- added R66, R67: 10K, SparkFun-Resistors:RESISTOR0805
Connections:
- new net N$47: Q3.S, R67.1, RPI-CM1G$1.GPIO14
- net +3V3: now also Q3.G, R67.2
- net +5V: now also R66.2
- net D2: now also Q3.D, R66.1
Changed lines of the file:
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@@
 <part name="P+29" library="supply1" library_urn="urn:adsk.eagle:library:371" deviceset="+5V" device=""/>
 <part name="GND3" library="supply1" library_urn="urn:adsk.eagle:library:371" deviceset="GND" device=""/>
+<part name="Q3" library="SparkFun" deviceset="MOSFET-NCHANNEL" device="SMD" value="BSS138"/>
+<part name="R66" library="SparkFun-Resistors" library_urn="urn:adsk.eagle:library:532" deviceset="RESISTOR" device="0805" package3d_urn="urn:adsk.eagle:package:39651/1" value="10K"/>
+<part name="R67" library="SparkFun-Resistors" library_urn="urn:adsk.eagle:library:532" deviceset="RESISTOR" device="0805" package3d_urn="urn:adsk.eagle:package:39651/1" value="10K"/>
+<part name="P+42" library="supply1" library_urn="urn:adsk.eagle:library:371" deviceset="+5V" device=""/>
+<part name="+3V4" library="supply1" library_urn="urn:adsk.eagle:library:371" deviceset="+3V3" device=""/>
+<part name="JP1" library="pinhead" library_urn="urn:adsk.eagle:library:325" deviceset="PINHD-2X20" device="" package3d_urn="urn:adsk.eagle:package:22443/2"/>
 </parts>
 <sheets>
@@
 <instance part="GND3" gate="1" x="203.2" y="137.16" smashed="yes" rot="R270">
 <attribute name="VALUE" x="200.66" y="139.7" size="1.778" layer="96" rot="R270"/>
+</instance>
+<instance part="Q3" gate="G$1" x="50.8" y="-2.54" smashed="yes" rot="R90">
+<attribute name="NAME" x="54.61" y="-7.366" size="1.778" layer="95" rot="R180"/>
+<attribute name="VALUE" x="56.134" y="3.048" size="1.778" layer="96" rot="R180"/>
+</instance>
+<instance part="R66" gate="G$1" x="43.18" y="2.54" smashed="yes" rot="R90">
+<attribute name="NAME" x="41.656" y="2.54" size="1.778" layer="95" font="vector" rot="R90" align="bottom-center"/>
+<attribute name="VALUE" x="44.704" y="2.54" size="1.778" layer="96" font="vector" rot="R90" align="top-center"/>
+</instance>
+<instance part="R67" gate="G$1" x="60.96" y="-7.62" smashed="yes" rot="R270">
+<attribute name="NAME" x="62.484" y="-7.62" size="1.778" layer="95" font="vector" rot="R270" align="bottom-center"/>
+<attribute name="VALUE" x="59.436" y="-7.62" size="1.778" layer="96" font="vector" rot="R270" align="top-center"/>
+</instance>
+<instance part="P+42" gate="1" x="43.18" y="12.7" smashed="yes">
+<attribute name="VALUE" x="40.64" y="7.62" size="1.778" layer="96" rot="R90"/>
+</instance>
+<instance part="+3V4" gate="G$1" x="68.58" y="-7.62" smashed="yes">
+<attribute name="VALUE" x="66.04" y="-12.7" size="1.778" layer="96" rot="R90"/>
+</instance>
+<instance part="JP1" gate="A" x="185.42" y="83.82" smashed="yes">
+<attribute name="NAME" x="179.07" y="109.855" size="1.778" layer="95"/>
+<attribute name="VALUE" x="179.07" y="53.34" size="1.778" layer="96"/>
 </instance>
 </instances>
@@
 <wire x1="149.86" y1="33.02" x2="160.02" y2="33.02" width="0.1524" layer="91"/>
 </segment>
+<segment>
+<pinref part="R67" gate="G$1" pin="2"/>
+<pinref part="+3V4" gate="G$1" pin="+3V3"/>
+<wire x1="60.96" y1="-12.7" x2="68.58" y2="-12.7" width="0.1524" layer="91"/>
+<wire x1="68.58" y1="-12.7" x2="68.58" y2="-10.16" width="0.1524" layer="91"/>
+<pinref part="Q3" gate="G$1" pin="G"/>
+<wire x1="50.8" y1="-10.16" x2="50.8" y2="-12.7" width="0.1524" layer="91"/>
+<wire x1="50.8" y1="-12.7" x2="60.96" y2="-12.7" width="0.1524" layer="91"/>
+<junction x="60.96" y="-12.7"/>
+</segment>
 </net>
 <net name="+5V" class="0">
@@
 <wire x1="259.08" y1="193.04" x2="264.16" y2="193.04" width="0.1524" layer="91"/>
 </segment>
+<segment>
+<pinref part="R66" gate="G$1" pin="2"/>
+<pinref part="P+42" gate="1" pin="+5V"/>
+<wire x1="43.18" y1="7.62" x2="43.18" y2="10.16" width="0.1524" layer="91"/>
+</segment>
 </net>
 <net name="D4" class="0">
@@
 <segment>
 <pinref part="U1" gate="A" pin="PD2"/>
-<wire x1="2.54" y1="-2.54" x2="15.24" y2="-2.54" width="0.1524" layer="91"/>
 <label x="5.08" y="-2.54" size="1.778" layer="95"/>
+<pinref part="R66" gate="G$1" pin="1"/>
+<pinref part="Q3" gate="G$1" pin="D"/>
+<wire x1="43.18" y1="-2.54" x2="45.72" y2="-2.54" width="0.1524" layer="91"/>
+<wire x1="2.54" y1="-2.54" x2="43.18" y2="-2.54" width="0.1524" layer="91"/>
+<junction x="43.18" y="-2.54"/>
 </segment>
 </net>
@@
 </segment>
 </net>
+<net name="N$47" class="0">
+<segment>
+<pinref part="Q3" gate="G$1" pin="S"/>
+<pinref part="R67" gate="G$1" pin="1"/>
+<wire x1="55.88" y1="-2.54" x2="60.96" y2="-2.54" width="0.1524" layer="91"/>
+<pinref part="RPI-CM1" gate="G$1" pin="GPIO14"/>
+<wire x1="88.9" y1="68.58" x2="60.96" y2="68.58" width="0.1524" layer="91"/>
+<wire x1="60.96" y1="68.58" x2="60.96" y2="-2.54" width="0.1524" layer="91"/>
+<junction x="60.96" y="-2.54"/>
+</segment>
+</net>
